Commit message: wip

File: models/vehicles/SEP/SEP_ship.urdf (robot description, URDF)
Before this commit: robot SEP_ship, 8 links, 6 joints
Links:
- added link support1; visual mesh filename=meshes/support1.glb
- added link support2; visual mesh filename=meshes/support2.glb
Joints:
- added joint support1: type fixed, parent base_link, child support1, origin xyz=8.9 -26.1 11.85
- added joint support2: type revolute, parent support1, child support2, origin xyz=-9.48 -3.85 0.0, axis 1 0 0, limit lower=-1.75 upper=1.75

Commit message: update model data

File: models/vehicles/SEP/SEP_ship.urdf (robot description, URDF)
Before this commit: robot SEP_ship, 10 links, 8 joints
Joints:
- joint crane_arm1: limit lower=-1.3 upper=0.12 -> lower=-1.5 upper=0.12
